File: Board/clock_1hz.kicad_sch (KiCad schematic)
At the start: 7 parts, among them U2 4040, U4 CD4060BE, Y1 32.768KHz

Commit message: fix 3.3v regulator footprint
Parts:
- C1, C2: footprint Capacitor_THT:C_Disc_D5.1mm_W3.2mm_P5.00mm -> Capacitor_THT:C_Disc_D3.0mm_W1.6mm_P2.50mm
Changed lines of the file:
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@@
       (effects (font (size 1.27 1.27)) (justify left))
     )
-    (property "Footprint" "Capacitor_THT:C_Disc_D5.1mm_W3.2mm_P5.00mm" (at 51.7652 71.12 0)
+    (property "Footprint" "Capacitor_THT:C_Disc_D3.0mm_W1.6mm_P2.50mm" (at 51.7652 71.12 0)
       (effects (font (size 1.27 1.27)) hide)
     )
@@
       (effects (font (size 1.27 1.27)) (justify left))
     )
-    (property "Footprint" "Capacitor_THT:C_Disc_D5.1mm_W3.2mm_P5.00mm" (at 64.4652 71.12 0)
+    (property "Footprint" "Capacitor_THT:C_Disc_D3.0mm_W1.6mm_P2.50mm" (at 64.4652 71.12 0)
       (effects (font (size 1.27 1.27)) hide)
     )
