File: Board/clock_1hz.kicad_sch (KiCad schematic)
At the start: 7 parts, among them U2 4040, U4 CD4060BE, Y1 32.768KHz

Commit message: make power circuit from 120v mains
Parts:
- removed C1, C2: 10pF, Capacitor_THT:C_Disc_D3.0mm_W1.6mm_P2.50mm, symbol Device:C
- removed R1: 330K, Resistor_THT:R_Axial_DIN0204_L3.6mm_D1.6mm_P7.62mm_Horizontal, symbol Device:R
- removed R2: 10M, Resistor_THT:R_Axial_DIN0204_L3.6mm_D1.6mm_P7.62mm_Horizontal, symbol Device:R
- removed U2: 4040, Package_DIP:DIP-16_W7.62mm_Socket, symbol 4xxx:4040
- removed U4: CD4060BE, Package_DIP:DIP-16_W7.62mm_Socket, symbol CD4060BE:CD4060BE
- removed Y1: 32.768KHz, Crystal:Crystal_C26-LF_D2.1mm_L6.5mm_Horizontal, symbol Device:Crystal
