File: Board/interface.kicad_sch (KiCad schematic)
At the start: 24 parts, among them SW1 SW_Push, SW2 SW_SPST_LED, SW3 SW_Push, U3 4069, U5 4069

Commit message: make power circuit from 120v mains
Parts:
- removed C3, C4, C5 (x3): 100nF, Capacitor_THT:C_Disc_D5.1mm_W3.2mm_P5.00mm, symbol Device:C
- removed R25 (x4), R3, R4, R9 (x3): 10K, Resistor_THT:R_Axial_DIN0204_L3.6mm_D1.6mm_P7.62mm_Horizontal, symbol Device:R
- removed SW1, SW3 (x3): SW_Push, Connector_JST:JST_XH_B2B-XH-A_1x02_P2.50mm_Vertical, symbol Switch:SW_Push
- removed SW2: SW_SPST_LED, Connector_JST:JST_XH_B3B-XH-A_1x03_P2.50mm_Vertical, symbol Switch:SW_SPST_LED
- removed U3 (x4), U5: 4069, Package_DIP:DIP-14_W7.62mm_Socket, symbol 4xxx_IEEE:4069
