File: Board/logic.kicad_sch (KiCad schematic)
At the start: 3 parts, among them U10 4071, U3 4081, U6 4071

Commit message: make power circuit from 120v mains
Parts:
- removed U10, U6: 4071, Package_DIP:DIP-14_W7.62mm_Socket, symbol 4xxx_IEEE:4071
- removed U3: 4081, Package_DIP:DIP-14_W7.62mm_Socket, symbol 4xxx_IEEE:4081
